File: Positron.kicad_sch (KiCad schematic)
At the start: 114 parts, among them CN1 GT-3321667P-01, J1 USB_C_Receptacle_USB2.0_16P, J2 Conn_01x04_Socket, J3 AudioJack3_SwitchTR, J4 PJ-603, J5 PJ-603, Q1 DMG1012T, SW1 TS-1187A-B-A-B, SW2 TS-1187A-B-A-B, U1 CS43198-CNZ, U10 SSM2019BRNZ, U2 TPS7A2036DBV, U3 TPS7A2018DBV, U4 STM32H743VITx, U5 RT6150AGQW, U6 OPA4134, U7 LM2776DBVR, U8 CS5361, U9 SSM2019BRNZ, Y1 Crystal_GND24

Commit message: fix balanced mic input
Parts:
- removed R18, R20: 400R, Resistor_SMD:R_0402_1005Metric, symbol Device:R_Small
Connections:
- net at J4.4: now also U9.2 (-IN)
- net at U10.2 (-IN): now also J5.4
Changed lines of the file:
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@@
 	(wire
 		(pts
+			(xy 66.04 234.95) (xy 66.04 231.14)
+		)
+		(stroke
+			(width 0)
+			(type default)
+		)
+	)
+	(wire
+		(pts
 			(xy 110.49 140.97) (xy 110.49 143.51)
 		)
@@
 	(wire
 		(pts
-			(xy 71.12 236.22) (xy 71.12 229.87)
-		)
-		(stroke
-			(width 0)
-			(type default)
-		)
-	)
-	(wire
-		(pts
 			(xy 273.05 138.43) (xy 281.94 138.43)
 		)
@@
 	(wire
 		(pts
-			(xy 71.12 190.5) (xy 71.12 184.15)
-		)
-		(stroke
-			(width 0)
-			(type default)
-		)
-	)
-	(wire
-		(pts
 			(xy 76.2 139.7) (xy 76.2 142.24)
 		)
@@
 	(wire
 		(pts
+			(xy 57.15 234.95) (xy 66.04 234.95)
+		)
+		(stroke
+			(width 0)
+			(type default)
+		)
+	)
+	(wire
+		(pts
 			(xy 156.21 99.06) (xy 160.02 99.06)
 		)
@@
 	(wire
 		(pts
+			(xy 76.2 231.14) (xy 76.2 229.87)
+		)
+		(stroke
+			(width 0)
+			(type default)
+		)
+	)
+	(wire
+		(pts
 			(xy 179.07 231.14) (xy 185.42 231.14)
 		)
@@
 	(wire
 		(pts
+			(xy 76.2 185.42) (xy 76.2 184.15)
+		)
+		(stroke
+			(width 0)
+			(type default)
+		)
+	)
+	(wire
+		(pts
 			(xy 93.98 184.15) (xy 95.25 184.15)
 		)
@@
 	(wire
 		(pts
-			(xy 71.12 229.87) (xy 76.2 229.87)
-		)
-		(stroke
-			(width 0)
-			(type default)
-		)
-	)
-	(wire
-		(pts
 			(xy 57.15 227.33) (xy 62.23 227.33)
 		)
@@
 	(wire
 		(pts
+			(xy 66.04 189.23) (xy 66.04 185.42)
+		)
+		(stroke
+			(width 0)
+			(type default)
+		)
+	)
+	(wire
+		(pts
 			(xy 82.55 106.68) (xy 82.55 127)
 		)
@@
 	(wire
 		(pts
+			(xy 66.04 185.42) (xy 76.2 185.42)
+		)
+		(stroke
+			(width 0)
+			(type default)
+		)
+	)
+	(wire
+		(pts
 			(xy 59.69 130.81) (xy 59.69 152.4)
 		)
@@
 	(wire
 		(pts
-			(xy 71.12 184.15) (xy 76.2 184.15)
-		)
-		(stroke
-			(width 0)
-			(type default)
-		)
-	)
-	(wire
-		(pts
 			(xy 69.85 189.23) (xy 76.2 189.23)
 		)
@@
 	(wire
 		(pts
+			(xy 57.15 189.23) (xy 66.04 189.23)
+		)
+		(stroke
+			(width 0)
+			(type default)
+		)
+	)
+	(wire
+		(pts
 			(xy 205.74 100.33) (xy 205.74 97.79)
 		)
@@
 	(wire
 		(pts
+			(xy 66.04 231.14) (xy 76.2 231.14)
+		)
+		(stroke
+			(width 0)
+			(type default)
+		)
+	)
+	(wire
+		(pts
 			(xy 138.43 157.48) (xy 138.43 167.64)
 		)
@@
 	)
 	(symbol
-		(lib_id "Device:R_Small")
-		(at 71.12 193.04 0)
-		(unit 1)
-		(body_style 1)
-		(exclude_from_sim no)
-		(in_bom yes)
-		(on_board yes)
-		(in_pos_files yes)
-		(dnp no)
-		(fields_autoplaced yes)
-		(property "Reference" "R18"
-			(at 73.66 191.7699 0)
-			(show_name no)
-			(do_not_autoplace no)
-			(effects
-				(font
-					(size 1.016 1.016)
-				)
-				(justify left)
-			)
-		)
-		(property "Value" "400R"
-			(at 73.66 194.3099 0)
-			(show_name no)
-			(do_not_autoplace no)
-			(effects
-				(font
-					(size 1.27 1.27)
-				)
-				(justify left)
-			)
-		)
-		(property "Footprint" "Resistor_SMD:R_0402_1005Metric"
-			(at 71.12 193.04 0)
-			(hide yes)
-			(show_name no)
-			(do_not_autoplace no)
-			(effects
-				(font
-					(size 1.27 1.27)
-				)
-			)
-		)
-		(property "Datasheet" ""
-			(at 71.12 193.04 0)
-			(hide yes)
-			(show_name no)
-			(do_not_autoplace no)
-			(effects
-				(font
-					(size 1.27 1.27)
-				)
-			)
-		)
-		(property "Description" "Resistor, small symbol"
-			(at 71.12 193.04 0)
-			(hide yes)
-			(show_name no)
-			(do_not_autoplace no)
-			(effects
-				(font
-					(size 1.27 1.27)
-				)
-			)
-		)
-		(pin "1"
-		)
-		(pin "2"
-		)
-		(instances
-			(project "Positron"
-				(path "/4d609ffc-7c1c-4898-8af9-f7815c412743"
-					(reference "R18")
-					(unit 1)
-				)
-			)
-		)
-	)
-	(symbol
 		(lib_id "power:VBUS")
 		(at 99.06 184.15 0)
@@
 					(unit 1)
 				)
-			)
-		)
-	)
-	(symbol
-		(lib_id "Device:R_Small")
-		(at 71.12 238.76 0)
-		(unit 1)
-		(body_style 1)
-		(exclude_from_sim no)
-		(in_bom yes)
-		(on_board yes)
-		(in_pos_files yes)
-		(dnp no)
-		(fields_autoplaced yes)
-		(property "Reference" "R20"
-			(at 73.66 237.4899 0)
-			(show_name no)
-			(do_not_autoplace no)
-			(effects
-				(font
-					(size 1.016 1.016)
-				)
-				(justify left)
-			)
-		)
-		(property "Value" "400R"
-			(at 73.66 240.0299 0)
-			(show_name no)
-			(do_not_autoplace no)
-			(effects
-				(font
-					(size 1.27 1.27)
-				)
-				(justify left)
-			)
-		)
-		(property "Footprint" "Resistor_SMD:R_0402_1005Metric"
-			(at 71.12 238.76 0)
-			(hide yes)
-			(show_name no)
-			(do_not_autoplace no)
-			(effects
-				(font
-					(size 1.27 1.27)
-				)
-			)
-		)
-		(property "Datasheet" ""
-			(at 71.12 238.76 0)
-			(hide yes)
-			(show_name no)
-			(do_not_autoplace no)
-			(effects
-				(font
-					(size 1.27 1.27)
-				)
-			)
-		)
-		(property "Description" "Resistor, small symbol"
-			(at 71.12 238.76 0)
-			(hide yes)
-			(show_name no)
-			(do_not_autoplace no)
-			(effects
-				(font
-					(size 1.27 1.27)
-				)
-			)
-		)
-		(pin "1"
-		)
-		(pin "2"
-		)
-		(instances
-			(project "Positron"
-				(path "/4d609ffc-7c1c-4898-8af9-f7815c412743"
-					(reference "R20")
-					(unit 1)
-				)

Commit message: separate GND planes and fill copper zone
Parts:
- added R18: 0R, Resistor_SMD:R_0402_1005Metric, symbol Device:R_Small
Connections:
- net GND: now also R18.1; no longer C10.2, C11.2, C12.2, C45.2, C46.2, C48.1, C49.2, C50.2, C51.1, C52.2, C53.1, C8.1, C9.1, CN1.1 (GND), CN1.11 (ep), CN1.12 (ep), CN1.9 (SW), J3.S, J4.2, J5.2, U1.19 (GNDCP), U1.8 (GNDA), U10.5 (REF), U7.2 (GND), U9.5 (REF)
- new net GNDA: C10.2, C11.2, C12.2, C45.2, C46.2, C48.1, C49.2, C50.2, C51.1, C52.2, C53.1, C8.1, C9.1, CN1.1 (GND), CN1.11 (ep), CN1.12 (ep), CN1.9 (SW), J3.S, J4.2, J5.2, R18.2, U1.19 (GNDCP), U1.8 (GNDA), U10.5 (REF), U7.2 (GND), U9.5 (REF)
