File: Resonance.kicad_pcb (KiCad board)
At the start: 4 copper layers, 104.3 x 34.2 mm, 123 parts, among them CN1 GT-3321667P-01, J1 USB_C_Receptacle_USB2.0_16P, J2 Conn_01x04_Socket, J3 AudioJack3_SwitchTR, SW1 TS-1187A-B-A-B, SW2 TS-1187A-B-A-B, U1 STM32F411CEUx, U10 OPA1622, U11 TPS63070RNMR, U12 TPS7A2050PDQN, U2 W25Q32RVXHJQ TR, U3 TPS7A2033PDBV, U4 CS43198-CNZ, U5 TPS7A2036PDBV, U6 TPS7A2018PDBV, U7 OPA1612AxD, U8 LM2776DBVR, U9 OPA1622, Y1 25MHz 9pF, Y2 32.768K 6pF

Commit message: add readme
Other:
- outline, holes or cut-outs redrawn
- board text added: "RESONANCE"
